Commit message: change name

File: src/mini_project/robots/argos.urdf.xacro (robot description, xacro)
@@ -37,8 +37,8 @@
         <material>Gazebo/FlatBlack</material>
     </gazebo>
-    <xacro:argus_leg leg="LF"/>
-    <xacro:argus_leg leg="RF"/>
-    <xacro:argus_leg leg="LH"/>
-    <xacro:argus_leg leg="RH"/>
+    <xacro:argos_leg leg="LF"/>
+    <xacro:argos_leg leg="RF"/>
+    <xacro:argos_leg leg="LH"/>
+    <xacro:argos_leg leg="RH"/>
     <xacro:include filename="$(find mini_project)/robots/manipulator.urdf.xacro"/>
     <xacro:manipulator base_name="base_link"/>

File: src/mini_project/robots/legs.urdf.xacro (robot description, xacro)
@@ -1,5 +1,5 @@
 <?xml version="1.0"?>
 <robot xmlns:xacro="http://www.ros.org/wiki/xacro">
-    <xacro:macro name="argus_leg" params="leg ">
+    <xacro:macro name="argos_leg" params="leg ">
         <xacro:if value="${leg == 'RF'}">
             <xacro:property name="side" value = "-1"/>
