Commit message: changes because of upgrade

File: src/mini_project/robots/accessories.urdf.xacro (robot description, xacro)
@@ -70,5 +70,5 @@
                 </image>
                 <clip>
-                <near>0.2</near>
+                <near>0.3</near>
                 <far>20</far>
                 </clip>
@@ -76,5 +76,5 @@
                 <type>gaussian</type>
                 <mean>0.0</mean>
-                <stddev>0.007</stddev>
+                <stddev>0.004</stddev>
                 </noise>
             </camera>
@@ -90,5 +90,5 @@
                 </image>
                 <clip>
-                <near>0.2</near>
+                <near>0.3</near>
                 <far>20</far>
                 </clip>
@@ -96,5 +96,5 @@
                 <type>gaussian</type>
                 <mean>0.0</mean>
-                <stddev>0.007</stddev>
+                <stddev>0.004</stddev>
                 </noise>
             </camera>
@@ -105,5 +105,5 @@
                 <imageTopicName>image_raw</imageTopicName>
                 <cameraInfoTopicName>camera_info</cameraInfoTopicName>
-                <frameName>camera_center</frameName>
+                <frameName>left_camera_optical_frame</frameName>
                 <!--<rightFrameName>right_camera_optical_frame</rightFrameName>-->
                 <hackBaseline>0.07</hackBaseline>
@@ -116,28 +116,4 @@
             </sensor>
         </gazebo>
-        <gazebo>
-            <plugin name="imu_controller" filename="libhector_gazebo_ros_imu.so">
-                <updateRate>50.0</updateRate>
-                <bodyName>imu_link</bodyName>
-                <topicName>imu/data</topicName>
-                <accelDrift>0.005 0.005 0.005</accelDrift>
-                <accelGaussianNoise>0.005 0.005 0.005</accelGaussianNoise>
-                <rateDrift>0.005 0.005 0.005 </rateDrift>
-                <rateGaussianNoise>0.005 0.005 0.005 </rateGaussianNoise>
-                <headingDrift>0.005</headingDrift>
-                <headingGaussianNoise>0.005</headingGaussianNoise>
-            </plugin>
-        </gazebo>
-        <link name="imu_link">
-            <inertial>
-                <mass value="0.001"/>
-                <origin xyz="0 0 0" rpy="0 0 0"/>
-                <inertia ixx="1e-09" ixy="0.0" ixz="0.0" iyy="1e-09" iyz="0.0" izz="1e-09"/>
-            </inertial>
-        </link>
-        <joint name="imu_joint" type="fixed">
-            <parent link="${base_name}" />
-            <child link="imu_link" />
-        </joint>
     </xacro:macro>
 </robot>

File: src/mini_project/robots/argos.urdf (robot description, URDF)
Before this commit: robot argos, 25 links, 24 joints
Links:
- removed link argos/base_link
- removed link imu_link
- added link base_link; collision mesh filename=package://mini_project/meshes/body.dae scale=0.001 0.001 0.001; visual mesh filename=package://mini_project/meshes/body.dae scale=0.001 0.001 0.001
Joints:
- removed joint argos/base_link_to_manipulator_joint
- removed joint imu_joint
- added joint base_link_to_manipulator_joint: type fixed, parent base_link, child manipulator_joint, origin xyz=0.0 0.0 0.13
- joint LF_hip_joint: parent argos/base_link -> base_link
- joint LH_hip_joint: parent argos/base_link -> base_link
- joint RF_hip_joint: parent argos/base_link -> base_link
- joint RH_hip_joint: parent argos/base_link -> base_link
- joint base_link_to_base_inertia: parent argos/base_link -> base_link
- joint camera_center_joint: parent argos/base_link -> base_link

File: src/mini_project/robots/argos.urdf.xacro (robot description, xacro)
@@ -4,5 +4,5 @@
     <xacro:property name="namespace" value="argos" />
     <xacro:include filename="$(find mini_project)/robots/robot_properties.urdf.xacro"/>
-    <link name="${namespace}/base_link">
+    <link name="base_link">
         <visual>
             <geometry>
@@ -28,5 +28,5 @@
     </link>
     <joint name="base_link_to_base_inertia" type="fixed">
-        <parent link="${namespace}/base_link"/>
+        <parent link="base_link"/>
         <child link="base_inertia"/>
         <origin rpy="0 0 0" xyz="0 0 0"/>
@@ -34,6 +34,6 @@
     <xacro:include filename="$(find mini_project)/robots/legs.urdf.xacro"/>
     <xacro:include filename="$(find mini_project)/robots/accessories.urdf.xacro"/>
-    <xacro:accessories base_name = "${namespace}/base_link"/>
-    <gazebo reference="${namespace}/base_link">
+    <xacro:accessories base_name = "base_link"/>
+    <gazebo reference="base_link">
         <material>Gazebo/FlatBlack</material>
     </gazebo>
@@ -43,10 +43,10 @@
     <xacro:argos_leg leg="RH"/>
     <xacro:include filename="$(find mini_project)/robots/manipulator.urdf.xacro"/>
-    <xacro:manipulator base_name="${namespace}/base_link"/>
+    <xacro:manipulator base_name="base_link"/>
     <gazebo>
       <plugin name="p3d_base_controller" filename="libgazebo_ros_p3d.so">
             <alwaysOn>true</alwaysOn>
             <updateRate>10.0</updateRate>
-            <bodyName>argos/base_link</bodyName>
+            <bodyName>base_link</bodyName>
             <topicName>odom/ground_truth</topicName>
             <gaussianNoise>0.01</gaussianNoise>
@@ -58,5 +58,4 @@
     <gazebo>
       <plugin filename="libgazebo_ros_control.so" name="gazebo_ros_control">
-        <legacyModeNS>true</legacyModeNS>
         <robotNamespace>/argos</robotNamespace>
       </plugin>

File: src/mini_project/robots/legs.urdf.xacro (robot description, xacro)
@@ -99,5 +99,5 @@
         <link name="${leg}_foot"/>
         <joint name="${leg}_hip_joint" type="revolute">
-            <parent link="${namespace}/base_link"/>
+            <parent link="base_link"/>
             <child link="${leg}_hip"/>
             <axis xyz="1.0 0.0 0.0"/>

Commit message: changes to make imu work

File: src/mini_project/robots/accessories.urdf.xacro (robot description, xacro)
@@ -116,4 +116,29 @@
             </sensor>
         </gazebo>
+        <gazebo>
+            <plugin name="imu_controller" filename="libhector_gazebo_ros_imu.so">
+                <updateRate>50.0</updateRate>
+                <bodyName>imu_link</bodyName>
+                <topicName>imu/data</topicName>
+                <accelDrift>0.005 0.005 0.005</accelDrift>
+                <frameId>argos/base_link</frameId>
+                <accelGaussianNoise>0.005 0.005 0.005</accelGaussianNoise>
+                <rateDrift>0.005 0.005 0.005 </rateDrift>
+                <rateGaussianNoise>0.005 0.005 0.005 </rateGaussianNoise>
+                <headingDrift>0.005</headingDrift>
+                <headingGaussianNoise>0.005</headingGaussianNoise>
+            </plugin>
+        </gazebo>
+        <link name="imu_link">
+            <inertial>
+                <mass value="0.001"/>
+                <origin xyz="0 0 0" rpy="0 0 0"/>
+                <inertia ixx="1e-09" ixy="0.0" ixz="0.0" iyy="1e-09" iyz="0.0" izz="1e-09"/>
+            </inertial>
+        </link>
+        <joint name="imu_joint" type="fixed">
+            <parent link="${base_name}" />
+            <child link="imu_link" />
+        </joint>
     </xacro:macro>
 </robot>

File: src/mini_project/robots/argos.urdf (robot description, URDF)
Before this commit: robot argos, 24 links, 23 joints
Links:
- added link imu_link, mass 0.001
Joints:
- added joint imu_joint: type fixed, parent base_link, child imu_link

File: src/mini_project/robots/argos.urdf.xacro (robot description, xacro)
@@ -2,5 +2,4 @@
 <robot xmlns:xacro="http://www.ros.org/wiki/xacro" name="argos">
     <xacro:property name="pi" value="3.14159265358979" />
-    <xacro:property name="namespace" value="argos" />
     <xacro:include filename="$(find mini_project)/robots/robot_properties.urdf.xacro"/>
     <link name="base_link">
@@ -58,5 +57,5 @@
     <gazebo>
       <plugin filename="libgazebo_ros_control.so" name="gazebo_ros_control">
-        <robotNamespace>/argos</robotNamespace>
+        <legacyModeNS>true</legacyModeNS>
       </plugin>
    </gazebo>

Commit message: adding pointcloud_to_laserscan

File: src/mini_project/robots/accessories.urdf.xacro (robot description, xacro)
@@ -9,5 +9,5 @@
     <xacro:arg name="cam_pos_x"     default="0.31" />
     <xacro:arg name="cam_pos_y"     default="0.0" />
-    <xacro:arg name="cam_pos_z"     default="0.12" />
+    <xacro:arg name="cam_pos_z"     default="-0.12" />
     <xacro:arg name="cam_roll"      default="0.0" />
     <xacro:arg name="cam_pitch"     default="0.0" />
@@ -58,5 +58,5 @@
         <gazebo reference="camera_center">
             <sensor type="multicamera" name="stereo_camera">
-            <update_rate>30.0</update_rate>
+            <update_rate>50.0</update_rate>
             <camera name="left">
                 <pose>0 0.06 0 0 0 0</pose>
@@ -65,11 +65,11 @@
                 <diagonal_fov>2.0943951</diagonal_fov>
                 <image>
-                <width>1920</width>
-                <height>1080</height>
-                <format>B8G8R8</format>
+                <width>1280</width>
+                <height>720</height>
+                <format>R8G8B8</format>
                 </image>
                 <clip>
-                <near>0.3</near>
-                <far>20</far>
+                <near>0.02</near>
+                <far>300</far>
                 </clip>
                 <noise>
@@ -85,11 +85,11 @@
                 <diagonal_fov>2.0943951</diagonal_fov>
                 <image>
-                <width>1920</width>
-                <height>1080</height>
-                <format>B8G8R8</format>
+                <width>1280</width>
+                <height>720</height>
+                <format>R8G8B8</format>
                 </image>
                 <clip>
-                <near>0.3</near>
-                <far>20</far>
+                <near>0.02</near>
+                <far>300</far>
                 </clip>
                 <noise>

File: src/mini_project/robots/argos.urdf (robot description, URDF)
Before this commit: robot argos, 25 links, 24 joints
Joints:
- joint LF_hip_joint: limit lower=-3.14159265358979 upper=3.14159265358979 effort=150 velocity=10 -> lower=-3.14159265358979 upper=3.14159265358979 effort=250 velocity=1.0
- joint LF_lower_leg_joint: limit lower=-3.14159265358979 upper=3.14159265358979 effort=150 velocity=10 -> lower=-3.14159265358979 upper=3.14159265358979 effort=250 velocity=1.0
- joint LF_upper_leg_joint: limit lower=-3.14159265358979 upper=3.14159265358979 effort=150 velocity=10 -> lower=-3.14159265358979 upper=3.14159265358979 effort=250 velocity=1.0
- joint LH_hip_joint: limit lower=-3.14159265358979 upper=3.14159265358979 effort=150 velocity=10 -> lower=-3.14159265358979 upper=3.14159265358979 effort=250 velocity=1.0
- joint LH_lower_leg_joint: limit lower=-3.14159265358979 upper=3.14159265358979 effort=150 velocity=10 -> lower=-3.14159265358979 upper=3.14159265358979 effort=250 velocity=1.0
- joint LH_upper_leg_joint: limit lower=-3.14159265358979 upper=3.14159265358979 effort=150 velocity=10 -> lower=-3.14159265358979 upper=3.14159265358979 effort=250 velocity=1.0
- joint RF_hip_joint: limit lower=-3.14159265358979 upper=3.14159265358979 effort=150 velocity=10 -> lower=-3.14159265358979 upper=3.14159265358979 effort=250 velocity=1.0
- joint RF_lower_leg_joint: limit lower=-3.14159265358979 upper=3.14159265358979 effort=150 velocity=10 -> lower=-3.14159265358979 upper=3.14159265358979 effort=250 velocity=1.0
- joint RF_upper_leg_joint: limit lower=-3.14159265358979 upper=3.14159265358979 effort=150 velocity=10 -> lower=-3.14159265358979 upper=3.14159265358979 effort=250 velocity=1.0
- joint RH_hip_joint: limit lower=-3.14159265358979 upper=3.14159265358979 effort=150 velocity=10 -> lower=-3.14159265358979 upper=3.14159265358979 effort=250 velocity=1.0
- joint RH_lower_leg_joint: limit lower=-3.14159265358979 upper=3.14159265358979 effort=150 velocity=10 -> lower=-3.14159265358979 upper=3.14159265358979 effort=250 velocity=1.0
- joint RH_upper_leg_joint: limit lower=-3.14159265358979 upper=3.14159265358979 effort=150 velocity=10 -> lower=-3.14159265358979 upper=3.14159265358979 effort=250 velocity=1.0
- joint camera_center_joint: origin xyz=0.31 0.0 0.12 rpy=0.0 0.0 0.0 -> xyz=0.31 0.0 -0.12 rpy=0.0 0.0 0.0

File: src/mini_project/robots/legs.urdf.xacro (robot description, xacro)
@@ -89,10 +89,10 @@
         </link>
         <gazebo reference="${leg}_lower_leg">
-            <kp>10000000.0</kp>
+            <kp>1000000.0</kp>
             <kd>1.0</kd>
-            <mu1>0.9</mu1>
-            <mu2>0.9</mu2>
-            <minDepth>0.005</minDepth>
-            <maxContacts>1</maxContacts>
+            <mu1>0.8</mu1>
+            <mu2>0.8</mu2>
+            <maxVel>0.0</maxVel>
+            <minDepth>0.001</minDepth>
             <material>Gazebo/Red</material>
         </gazebo>
@@ -103,6 +103,5 @@
             <axis xyz="1.0 0.0 0.0"/>
             <origin xyz="${position_hip} 0.0 0.0"/>
-            <limit effort="150" lower="-${pi}" upper="${pi}" velocity="10" />
-      <dynamics damping="0.0" friction="0.0" />
+            <limit effort="250" lower="-${pi}" upper="${pi}" velocity="1.0" />
         </joint>
         <joint name="${leg}_upper_leg_joint" type="revolute">
@@ -111,6 +110,5 @@
             <axis xyz="0.0 1.0  0.0"/>
             <origin xyz="0.0 ${side*0.233} 0.0"/>
-            <limit effort="150" lower="-${pi}" upper="${pi}" velocity="10" />
-      <dynamics damping="0.0" friction="0.0" />
+            <limit effort="250" lower="-${pi}" upper="${pi}" velocity="1.0" />
         </joint>
         <joint name="${leg}_lower_leg_joint" type="revolute">
@@ -119,6 +117,5 @@
             <axis xyz="0.0 1.0  0.0"/>
             <origin xyz="0.0 0.0 -0.45"/>
-            <limit effort="150" lower="-${pi}" upper="${pi}" velocity="10" />
-      <dynamics damping="0.0" friction="0.0" />
+            <limit effort="250" lower="-${pi}" upper="${pi}" velocity="1.0" />
         </joint>
         <joint name="${leg}_foot_joint" type="fixed">
@@ -130,8 +127,7 @@
             <type>transmission_interface/SimpleTransmission</type>
             <joint name="${leg}_hip_joint">
-                <hardwareInterface>hardware_interface/EffortJointInterface</hardwareInterface>
+                <hardwareInterface>EffortJointInterface</hardwareInterface>
             </joint>
             <actuator name="${leg}_hip_joint_motor">
-                <hardwareInterface>hardware_interface/EffortJointInterface</hardwareInterface>
                 <mechanicalReduction>1</mechanicalReduction>
             </actuator>
@@ -140,8 +136,7 @@
             <type>transmission_interface/SimpleTransmission</type>
             <joint name="${leg}_upper_leg_joint">
-                <hardwareInterface>hardware_interface/EffortJointInterface</hardwareInterface>
+                <hardwareInterface>EffortJointInterface</hardwareInterface>
             </joint>
             <actuator name="${leg}_upper_leg_joint_motor">
-                <hardwareInterface>hardware_interface/EffortJointInterface</hardwareInterface>
                 <mechanicalReduction>1</mechanicalReduction>
             </actuator>
@@ -150,8 +145,7 @@
             <type>transmission_interface/SimpleTransmission</type>
             <joint name="${leg}_lower_leg_joint">
-                <hardwareInterface>hardware_interface/EffortJointInterface</hardwareInterface>
+                <hardwareInterface>EffortJointInterface</hardwareInterface>
             </joint>
             <actuator name="${leg}_lower_joint_motor">
-                <hardwareInterface>hardware_interface/EffortJointInterface</hardwareInterface>
                 <mechanicalReduction>1</mechanicalReduction>
             </actuator>

File: src/mini_project/robots/robot_properties.urdf.xacro (robot description, xacro)
@@ -17,8 +17,8 @@
     <xacro:property name="body_center_of_mass" value = "0 0 -0.00722624877"/>
     <xacro:property name="ixx_leg_roll" value = "0.01771591024568"/>
-    <xacro:property name="ixy_leg_roll" value = "-0.00071891013320"/>
-    <xacro:property name="ixz_leg_roll" value = "0.00000000005151"/>
+    <xacro:property name="ixy_leg_roll" value = "0.0"/>
+    <xacro:property name="ixz_leg_roll" value = "0.0"/>
     <xacro:property name="iyy_leg_roll" value = "0.00540298667217"/>
-    <xacro:property name="iyz_leg_roll" value = "0.00000000016635"/>
+    <xacro:property name="iyz_leg_roll" value = "0.0"/>
     <xacro:property name="izz_leg_roll" value = "0.01761332943090"/>
     <xacro:property name="leg_roll_mass" value = "2.33840380"/>
@@ -39,5 +39,5 @@
     <xacro:property name="ixx_lower_leg" value = "0.0938058"/>
     <xacro:property name="ixy_lower_leg" value = "0.0"/>
-    <xacro:property name="ixz_lower_leg" value = "-0.00320577"/>
+    <xacro:property name="ixz_lower_leg" value = "0.0"/>
     <xacro:property name="iyy_lower_leg" value = "0.09632913"/>
     <xacro:property name="iyz_lower_leg" value = "0.0"/>
@@ -49,24 +49,24 @@
     <xacro:property name="lower_leg_center_of_mass" value = "${lower_leg_center_x} ${lower_leg_center_y} ${lower_leg_center_z}"/>
     <xacro:property name="ixx_man_base" value = "0.00592368152307"/>
-    <xacro:property name="ixy_man_base" value = "-0.00000002959529"/>
-    <xacro:property name="ixz_man_base" value = "0.00000000508195"/>
+    <xacro:property name="ixy_man_base" value = "0.0"/>
+    <xacro:property name="ixz_man_base" value = "0.0"/>
     <xacro:property name="iyy_man_base" value = "0.00455222665474"/>
-    <xacro:property name="iyz_man_base" value = "-0.00046066688062"/>
+    <xacro:property name="iyz_man_base" value = "0.0"/>
     <xacro:property name="izz_man_base" value = "0.00630165344962"/>
     <xacro:property name="man_base_mass" value = "1.63291158"/>
     <xacro:property name="man_base_center" value = "0.0001195 -0.01132600777 0.04996291284 "/>
     <xacro:property name="ixx_man_seg_1" value = "0.00029149081721"/>
-    <xacro:property name="ixy_man_seg_1" value = "0.00000011029091"/>
-    <xacro:property name="ixz_man_seg_1" value = "-0.00000000001180"/>
+    <xacro:property name="ixy_man_seg_1" value = "0.0"/>
+    <xacro:property name="ixz_man_seg_1" value = "0.0"/>
     <xacro:property name="iyy_man_seg_1" value = "0.00745356022911"/>
-    <xacro:property name="iyz_man_seg_1" value = "-0.00000000000194"/>
+    <xacro:property name="iyz_man_seg_1" value = "0.0"/>
     <xacro:property name="izz_man_seg_1" value = "0.00730622307390"/>
     <xacro:property name="man_seg_1_mass" value = "0.65721313"/>
     <xacro:property name="man_seg_1_center" value = "-0.12499144985 0.00000184653 0.0"/>
     <xacro:property name="ixx_man_seg_2" value = "0.00016867187941"/>
-    <xacro:property name="ixy_man_seg_2" value = "-0.00000000001369"/>
-    <xacro:property name="ixz_man_seg_2" value = "0.00000000184646"/>
+    <xacro:property name="ixy_man_seg_2" value = "0.0"/>
+    <xacro:property name="ixz_man_seg_2" value = "0.0"/>
     <xacro:property name="iyy_man_seg_2" value = "0.02041441059327"/>
-    <xacro:property name="iyz_man_seg_2" value = "0.00000000000093"/>
+    <xacro:property name="iyz_man_seg_2" value = "0.0"/>
     <xacro:property name="izz_man_seg_2" value = "0.02036185070001"/>
     <xacro:property name="man_seg_2_mass" value = "0.45716422"/>
