Commit message: adding ground_truth, pointcloud_to_laserscan,disparity_to_laserscan,depth_camera_to_laserscan and improving movement

File: src/mini_project/robots/accessories_depth.urdf.xacro (robot description, xacro)
@@ -57,4 +57,50 @@
     <link name="left_camera_optical_frame"/>
     <gazebo reference="left_camera_frame">
+        <sensor type="depth" name="openni_camera_camera">
+        <always_on>1</always_on>
+        <visualize>true</visualize>
+        <camera>
+            <horizontal_fov>1.91986218</horizontal_fov>
+            <vertical_fov>1.22173048</vertical_fov>
+            <diagonal_fov>2.0943951</diagonal_fov>
+            <image>
+                <width>1920</width>
+                <height>1080</height>
+                <format>R8G8B8</format>
+            </image>
+            <clip>
+                <near>0.1</near>
+                <far>25.0</far>
+            </clip>
+        </camera>
+        <plugin name="camera_plugin" filename="libgazebo_ros_openni_kinect.so">
+            <robotNamespace>argos</robotNamespace>
+            <baseline>0.2</baseline>
+            <alwaysOn>true</alwaysOn>
+            <!-- Keep this zero, update_rate in the parent <sensor> tag
+                will control the frame rate. -->
+            <updateRate>0.0</updateRate>
+            <cameraName>depth_camera</cameraName>
+            <imageTopicName>/depth/image_rect_color</imageTopicName>
+            <cameraInfoTopicName>/argos/depth/camera_info </cameraInfoTopicName>
+            <depthImageTopicName>/argos/depth/depth_registered</depthImageTopicName>
+            <depthImageCameraInfoTopicName>/argos/depth/image_raw/camera_info</depthImageCameraInfoTopicName>
+            <pointCloudTopicName>/argos/depth/point_cloud/cloud_registered </pointCloudTopicName>
+            <frameName>left_camera_optical_frame</frameName>
+            <pointCloudCutoff>0.4</pointCloudCutoff>
+            <!-- does nothing it seems
+            <pointCloudCutoffMax>20.0</pointCloudCutoffMax> -->
+            <distortionK1>0</distortionK1>
+            <distortionK2>0</distortionK2>
+            <distortionK3>0</distortionK3>
+            <distortionT1>0</distortionT1>
+            <distortionT2>0</distortionT2>
+            <CxPrime>0</CxPrime>
+            <Cx>0</Cx>
+            <Cy>0</Cy>
+            <focalLength>0</focalLength>
+            <hackBaseline>0</hackBaseline>
+        </plugin>
+        </sensor>
         <sensor type="multicamera" name="stereo_camera">
         <update_rate>30.0</update_rate>

File: src/mini_project/robots/argos_depth.urdf.xacro (robot description, xacro)
@@ -32,5 +32,5 @@
     </joint>
     <xacro:include filename="$(find mini_project)/robots/legs.urdf.xacro"/>
-    <xacro:include filename="$(find mini_project)/robots/accessories.urdf.xacro"/>
+    <xacro:include filename="$(find mini_project)/robots/accessories_depth.urdf.xacro"/>
     <xacro:accessories base_name = "base_link"/>
     <gazebo reference="base_link">

File: src/mini_project/robots/legs.urdf.xacro (robot description, xacro)
@@ -19,4 +19,9 @@
         </xacro:if>
         <xacro:property name="leg_roll_center_of_mass" value = "${side*leg_roll_center_x} ${side*leg_roll_center_y} ${leg_roll_center_z}"/>
+        <xacro:property name="toeOffset" value="0.0106"/>
+        <xacro:property name="toeStiffness" value="30000.0"/>
+        <xacro:property name="toeDamping" value="1000.0"/>
+        <xacro:property name="toeFriction" value="1.0"/>
+        <xacro:property name="toeLateralFriction" value="1.0"/>
         <link name="${leg}_leg_roll">
             <inertial>
@@ -45,5 +50,5 @@
         <link name="${leg}_upper_leg">
             <inertial>
-                <origin xyz = "${thigh_center_of_mass}"  rpy="0 0 0"/>
+                <origin xyz = "${thigh_center_of_mass}"  rpy="${pi/2} 0 ${pi/2}"/>
                 <mass value="${thigh_mass}" />
                 <inertia ixx="${ixx_thigh}" ixy="${side*ixy_thigh}" ixz="${ixz_thigh}"
@@ -69,5 +74,5 @@
         <link name="${leg}_lower_leg">
             <inertial>
-                <origin xyz = "${lower_leg_center_of_mass}" rpy="0 0 0"/>
+                <origin xyz = "${lower_leg_center_of_mass}" rpy="0 -0.2 0"/>
                 <mass value="${lower_leg_mass}" />
                 <inertia ixx="${ixx_lower_leg}" ixy="${ixy_lower_leg}" ixz="${ixz_lower_leg}"
@@ -79,5 +84,5 @@
                     <mesh filename="${path_to_lower_leg}" scale = "0.001 0.001 0.001"/>
                 </geometry>
-                <origin xyz="0 0.0 0" rpy="${pi/2} ${pi/2-0.182960291} 0"/>
+                <origin xyz="0 0.0 0" rpy="${pi/2} ${pi/2-0.2} 0"/>
             </visual>
             <collision>
@@ -85,12 +90,12 @@
                     <mesh filename="${path_to_lower_leg}" scale = "0.001 0.001 0.001"/>
                 </geometry>
-                <origin xyz="0 0.0 0" rpy="${pi/2} ${pi/2-0.182960291} 0"/>
+                <origin xyz="0 0.0 0" rpy="${pi/2} ${pi/2-0.2} 0"/>
             </collision>
         </link>
         <gazebo reference="${leg}_lower_leg">
-            <kp>1000000.0</kp>
+			<kp>100000.0</kp>
             <kd>1.0</kd>
-            <mu1>0.8</mu1>
-            <mu2>0.8</mu2>
+            <mu1>1.0</mu1>
+            <mu2>1.0</mu2>
             <maxVel>0.0</maxVel>
             <minDepth>0.001</minDepth>
@@ -103,5 +108,5 @@
             <axis xyz="1.0 0.0 0.0"/>
             <origin xyz="${position_hip} 0.0 0.0"/>
-            <limit effort="250" lower="-${pi}" upper="${pi}" velocity="1.0" />
+            <limit effort="250" lower="-${pi}" upper="${pi}" velocity="5.0" />
         </joint>
         <joint name="${leg}_upper_leg_joint" type="revolute">
@@ -110,5 +115,5 @@
             <axis xyz="0.0 1.0  0.0"/>
             <origin xyz="0.0 ${side*0.233} 0.0"/>
-            <limit effort="250" lower="-${pi}" upper="${pi}" velocity="1.0" />
+            <limit effort="250" lower="-${pi}" upper="${pi}" velocity="5.0" />
         </joint>
         <joint name="${leg}_lower_leg_joint" type="revolute">
@@ -117,15 +122,24 @@
             <axis xyz="0.0 1.0  0.0"/>
             <origin xyz="0.0 0.0 -0.45"/>
-            <limit effort="250" lower="-${pi}" upper="${pi}" velocity="1.0" />
+            <limit effort="250" lower="-${pi}" upper="${pi}" velocity="2.0" />
         </joint>
         <joint name="${leg}_foot_joint" type="fixed">
             <parent link="${leg}_lower_leg"/>
             <child link="${leg}_foot"/>
-            <origin xyz="-0.0 0.0 -0.61"/>
+            <origin xyz="0.0 0.0 -0.61"/>
         </joint>
+        <gazebo reference="${leg}_hip_joint">
+            <provideFeedback>true</provideFeedback>
+        </gazebo>
+        <gazebo reference="${leg}_upper_leg_joint">
+            <provideFeedback>true</provideFeedback>
+        </gazebo>
+        <gazebo reference="${leg}_lower_leg_joint">
+            <provideFeedback>true</provideFeedback>
+        </gazebo>
         <transmission name="${leg}_hip_joint_trans">
             <type>transmission_interface/SimpleTransmission</type>
             <joint name="${leg}_hip_joint">
-                <hardwareInterface>EffortJointInterface</hardwareInterface>
+            <hardwareInterface>hardware_interface/EffortJointInterface</hardwareInterface>
             </joint>
             <actuator name="${leg}_hip_joint_motor">
@@ -136,5 +150,5 @@
             <type>transmission_interface/SimpleTransmission</type>
             <joint name="${leg}_upper_leg_joint">
-                <hardwareInterface>EffortJointInterface</hardwareInterface>
+            <hardwareInterface>hardware_interface/EffortJointInterface</hardwareInterface>
             </joint>
             <actuator name="${leg}_upper_leg_joint_motor">
@@ -145,5 +159,5 @@
             <type>transmission_interface/SimpleTransmission</type>
             <joint name="${leg}_lower_leg_joint">
-                <hardwareInterface>EffortJointInterface</hardwareInterface>
+            <hardwareInterface>hardware_interface/EffortJointInterface</hardwareInterface>
             </joint>
             <actuator name="${leg}_lower_joint_motor">

File: src/mini_project/robots/robot_properties.urdf.xacro (robot description, xacro)
@@ -8,43 +8,43 @@
     <xacro:property name="path_to_manipulator_segment_1" value = "package://mini_project/meshes/manipulator_segment_1.dae"/>
     <xacro:property name="path_to_manipulator_segment_2" value = "package://mini_project/meshes/manipulator_segment_2.dae"/>
-    <xacro:property name="ixx_body" value = "0.47331170488629"/>
-    <xacro:property name="ixy_body" value = "0.0"/>
-    <xacro:property name="ixz_body" value = "0.0"/>
-    <xacro:property name="iyy_body" value = "1.92964600184763"/>
-    <xacro:property name="iyz_body" value = "0.0"/>
-    <xacro:property name="izz_body" value = "1.88984590052932"/>
-    <xacro:property name="body_mass" value = "44.88560358"/>
+    <xacro:property name="ixx_body" value = "0.47331170488628769"/>
+    <xacro:property name="ixy_body" value = "-0.00000001187694189"/>
+    <xacro:property name="ixz_body" value = "0.00000000000000003"/>
+    <xacro:property name="iyy_body" value = "1.92964600184763336"/>
+    <xacro:property name="iyz_body" value = "-0.00000000000000002"/>
+    <xacro:property name="izz_body" value = "1.88984590052932334"/>
+    <xacro:property name="body_mass" value = "44.88560357849"/>
     <xacro:property name="body_center_of_mass" value = "0 0 -0.00722624877"/>
-    <xacro:property name="ixx_leg_roll" value = "0.01771591024568"/>
-    <xacro:property name="ixy_leg_roll" value = "0.0"/>
-    <xacro:property name="ixz_leg_roll" value = "0.0"/>
-    <xacro:property name="iyy_leg_roll" value = "0.00540298667217"/>
-    <xacro:property name="iyz_leg_roll" value = "0.0"/>
-    <xacro:property name="izz_leg_roll" value = "0.01761332943090"/>
-    <xacro:property name="leg_roll_mass" value = "2.33840380"/>
+    <xacro:property name="ixx_leg_roll" value = "0.01771591024567954"/>
+    <xacro:property name="ixy_leg_roll" value = "-0.00071891013320325"/>
+    <xacro:property name="ixz_leg_roll" value = "0.00000000005150730"/>
+    <xacro:property name="iyy_leg_roll" value = "0.00540298667216859"/>
+    <xacro:property name="iyz_leg_roll" value = "0.00000000016635487"/>
+    <xacro:property name="izz_leg_roll" value = "0.01761332943089841"/>
+    <xacro:property name="leg_roll_mass" value = "2.33840380361"/>
     <xacro:property name="leg_roll_center_x" value = "0.00160346990"/>
     <xacro:property name="leg_roll_center_y" value = "0.19560047521"/>
     <xacro:property name="leg_roll_center_z" value = "0.0"/>
-    <xacro:property name="ixx_thigh" value = "0.07057863"/>
-    <xacro:property name="ixy_thigh" value = "0.0"/>
-    <xacro:property name="ixz_thigh" value = "0.0"/>
-    <xacro:property name="iyy_thigh" value = "0.07214686"/>
-    <xacro:property name="iyz_thigh" value = "0.0"/>
-    <xacro:property name="izz_thigh" value = "0.00313293"/>
-    <xacro:property name="thigh_mass" value = "2.90604712"/>
-    <xacro:property name="thigh_center_x" value = "0.0"/>
-    <xacro:property name="thigh_center_y" value = "0.0"/>
-    <xacro:property name="thigh_center_z" value = "-0.19777343"/>
+    <xacro:property name="ixx_thigh" value = "0.07057863001314926"/>
+    <xacro:property name="ixy_thigh" value = "0.00000000027932686"/>
+    <xacro:property name="ixz_thigh" value = "-0.00000000037129365"/>
+    <xacro:property name="iyy_thigh" value = "0.07214686311642775"/>
+    <xacro:property name="iyz_thigh" value = "-0.00000000697351520"/>
+    <xacro:property name="izz_thigh" value = "0.00313292947996250"/>
+    <xacro:property name="thigh_mass" value = "2.90604711841"/>
+    <xacro:property name="thigh_center_x" value = "-0.00000012465"/>
+    <xacro:property name="thigh_center_y" value = "0.00000008927"/>
+    <xacro:property name="thigh_center_z" value = "-0.19777343169"/>
     <xacro:property name="thigh_center_of_mass" value = "${thigh_center_x} ${thigh_center_y} ${thigh_center_z}"/>
-    <xacro:property name="ixx_lower_leg" value = "0.0938058"/>
-    <xacro:property name="ixy_lower_leg" value = "0.0"/>
-    <xacro:property name="ixz_lower_leg" value = "0.0"/>
-    <xacro:property name="iyy_lower_leg" value = "0.09632913"/>
-    <xacro:property name="iyz_lower_leg" value = "0.0"/>
-    <xacro:property name="izz_lower_leg" value = "0.00375697"/>
-    <xacro:property name="lower_leg_mass" value = "1.81736395"/>
-    <xacro:property name="lower_leg_center_x" value = "-0.02510293"/>
-    <xacro:property name="lower_leg_center_y" value = "0.0"/>
-    <xacro:property name="lower_leg_center_z" value = "-0.15457863"/>
+    <xacro:property name="ixx_lower_leg" value = "0.09079395557915390"/>
+    <xacro:property name="ixy_lower_leg" value = "-0.00000001255242645"/>
+    <xacro:property name="ixz_lower_leg" value = "0.01304754928405628"/>
+    <xacro:property name="iyy_lower_leg" value = "0.09510714803975490"/>
+    <xacro:property name="iyz_lower_leg" value = "-0.00000000639667712"/>
+    <xacro:property name="izz_lower_leg" value = "0.00552232540194871"/>
+    <xacro:property name="lower_leg_mass" value = "1.81736381294"/>
+    <xacro:property name="lower_leg_center_x" value = "-0.05466888228"/>
+    <xacro:property name="lower_leg_center_y" value = "0.00000002713"/>
+    <xacro:property name="lower_leg_center_z" value = "-0.15386388146"/>
     <xacro:property name="lower_leg_center_of_mass" value = "${lower_leg_center_x} ${lower_leg_center_y} ${lower_leg_center_z}"/>
     <xacro:property name="ixx_man_base" value = "0.00592368152307"/>
