Commit message: adding robot name

File: src/mini_project/robots/argos.urdf (robot description, URDF)
Before this commit: robot argos, 25 links, 24 joints
Links:
- removed link base_link
- added link argos/base_link; collision mesh filename=package://mini_project/meshes/body.dae scale=0.001 0.001 0.001; visual mesh filename=package://mini_project/meshes/body.dae scale=0.001 0.001 0.001
Joints:
- removed joint base_link_to_manipulator_joint
- added joint argos/base_link_to_manipulator_joint: type fixed, parent argos/base_link, child manipulator_joint, origin xyz=0.0 0.0 0.13
- joint LF_hip_joint: parent base_link -> argos/base_link
- joint LH_hip_joint: parent base_link -> argos/base_link
- joint RF_hip_joint: parent base_link -> argos/base_link
- joint RH_hip_joint: parent base_link -> argos/base_link
- joint base_link_to_base_inertia: parent base_link -> argos/base_link
- joint camera_center_joint: parent base_link -> argos/base_link
- joint imu_joint: parent base_link -> argos/base_link

File: src/mini_project/robots/argos.urdf.xacro (robot description, xacro)
@@ -2,6 +2,7 @@
 <robot xmlns:xacro="http://www.ros.org/wiki/xacro" name="argos">
     <xacro:property name="pi" value="3.14159265358979" />
+    <xacro:property name="namespace" value="argos" />
     <xacro:include filename="$(find mini_project)/robots/robot_properties.urdf.xacro"/>
-    <link name="base_link">
+    <link name="${namespace}/base_link">
         <visual>
             <geometry>
@@ -27,5 +28,5 @@
     </link>
     <joint name="base_link_to_base_inertia" type="fixed">
-        <parent link="base_link"/>
+        <parent link="${namespace}/base_link"/>
         <child link="base_inertia"/>
         <origin rpy="0 0 0" xyz="0 0 0"/>
@@ -33,6 +34,6 @@
     <xacro:include filename="$(find mini_project)/robots/legs.urdf.xacro"/>
     <xacro:include filename="$(find mini_project)/robots/accessories.urdf.xacro"/>
-    <xacro:accessories base_name = "base_link"/>
-    <gazebo reference="base_link">
+    <xacro:accessories base_name = "${namespace}/base_link"/>
+    <gazebo reference="${namespace}/base_link">
         <material>Gazebo/FlatBlack</material>
     </gazebo>
@@ -42,8 +43,21 @@
     <xacro:argos_leg leg="RH"/>
     <xacro:include filename="$(find mini_project)/robots/manipulator.urdf.xacro"/>
-    <xacro:manipulator base_name="base_link"/>
+    <xacro:manipulator base_name="${namespace}/base_link"/>
+    <gazebo>
+      <plugin name="p3d_base_controller" filename="libgazebo_ros_p3d.so">
+            <alwaysOn>true</alwaysOn>
+            <updateRate>10.0</updateRate>
+            <bodyName>argos/base_link</bodyName>
+            <topicName>odom/ground_truth</topicName>
+            <gaussianNoise>0.01</gaussianNoise>
+            <frameName>world</frameName>
+            <xyzOffsets>0 0 0</xyzOffsets>
+            <rpyOffsets>0 0 0</rpyOffsets>
+        </plugin>
+    </gazebo>
     <gazebo>
       <plugin filename="libgazebo_ros_control.so" name="gazebo_ros_control">
-         <legacyModeNS>true</legacyModeNS>
+        <legacyModeNS>true</legacyModeNS>
+        <robotNamespace>/argos</robotNamespace>
       </plugin>
    </gazebo>

File: src/mini_project/robots/legs.urdf.xacro (robot description, xacro)
@@ -99,5 +99,5 @@
         <link name="${leg}_foot"/>
         <joint name="${leg}_hip_joint" type="revolute">
-            <parent link="base_link"/>
+            <parent link="${namespace}/base_link"/>
             <child link="${leg}_hip"/>
             <axis xyz="1.0 0.0 0.0"/>

Commit message: adding stereo params

File: src/mini_project/robots/argos.urdf (robot description, URDF)
Before this commit: robot argos, 25 links, 24 joints
Links:
- removed link LF_hip
- removed link LH_hip
- removed link RF_hip
- removed link RH_hip
- removed link manipulator_joint
- added link LF_leg_roll, mass 2.3384038; collision mesh filename=package://mini_project/meshes/thigh.dae scale=0.001 0.001 0.001; visual mesh filename=package://mini_project/meshes/thigh.dae scale=0.001 0.001 0.001
- added link LH_leg_roll, mass 2.3384038; collision mesh filename=package://mini_project/meshes/thigh.dae scale=0.001 0.001 0.001; visual mesh filename=package://mini_project/meshes/thigh.dae scale=0.001 0.001 0.001
- added link RF_leg_roll, mass 2.3384038; collision mesh filename=package://mini_project/meshes/thigh.dae scale=0.001 0.001 0.001; visual mesh filename=package://mini_project/meshes/thigh.dae scale=0.001 0.001 0.001
- added link RH_leg_roll, mass 2.3384038; collision mesh filename=package://mini_project/meshes/thigh.dae scale=0.001 0.001 0.001; visual mesh filename=package://mini_project/meshes/thigh.dae scale=0.001 0.001 0.001
- added link manipulator_base, mass 1.63291158; collision mesh filename=package://mini_project/meshes/manipulator_joint.dae scale=0.001 0.001 0.001; visual mesh filename=package://mini_project/meshes/manipulator_joint.dae scale=0.001 0.001 0.001
Joints:
- removed joint base_link_to_manipulator_joint
- removed joint manipulator_joint_to_manipulator_segment_1
- added joint base_link_to_manipulator_base: type fixed, parent base_link, child manipulator_base, origin xyz=0.0 0.0 0.13
- added joint manipulator_base_to_manipulator_segment_1: type fixed, parent manipulator_base, child manipulator_segment_1, origin xyz=0.0 0.04 0.075 rpy=0 0 0
- joint LF_hip_joint: child LF_hip -> LF_leg_roll
- joint LF_upper_leg_joint: parent LF_hip -> LF_leg_roll
- joint LH_hip_joint: child LH_hip -> LH_leg_roll
- joint LH_upper_leg_joint: parent LH_hip -> LH_leg_roll
- joint RF_hip_joint: child RF_hip -> RF_leg_roll
- joint RF_upper_leg_joint: parent RF_hip -> RF_leg_roll
- joint RH_hip_joint: child RH_hip -> RH_leg_roll
- joint RH_upper_leg_joint: parent RH_hip -> RH_leg_roll

File: src/mini_project/robots/legs.urdf.xacro (robot description, xacro)
@@ -18,16 +18,16 @@
             <xacro:property name="position_hip" value = "-0.43"/>
         </xacro:if>
-        <xacro:property name="hip_center_of_mass" value = "${side*hip_center_x} ${side*hip_center_y} ${hip_center_z}"/>
-        <link name="${leg}_hip">
+        <xacro:property name="leg_roll_center_of_mass" value = "${side*leg_roll_center_x} ${side*leg_roll_center_y} ${leg_roll_center_z}"/>
+        <link name="${leg}_leg_roll">
             <inertial>
-                <origin xyz = "${hip_center_of_mass}"  rpy="0 0 0"/>
-                <mass value="${hip_mass}" />
-                <inertia ixx="${ixx_hip}" ixy="${ixy_hip}" ixz="${ixz_hip}"
-                     iyy="${iyy_hip}" iyz="${iyz_hip}"
-                     izz="${izz_hip}" />
+                <origin xyz = "${leg_roll_center_of_mass}"  rpy="0 0 0"/>
+                <mass value="${leg_roll_mass}" />
+                <inertia ixx="${ixx_leg_roll}" ixy="${ixy_leg_roll}" ixz="${ixz_leg_roll}"
+                     iyy="${iyy_leg_roll}" iyz="${iyz_leg_roll}"
+                     izz="${izz_leg_roll}" />
             </inertial>
             <visual>
                 <geometry>
-                    <mesh filename="${path_to_hip}" scale = "0.001 0.001 0.001"/>
+                    <mesh filename="${path_to_leg_roll}" scale = "0.001 0.001 0.001"/>
                 </geometry>
                 <origin xyz="0.0 0.0 0.0" rpy="${pi/2} 0.0 ${pi*side/2}" />
@@ -35,10 +35,10 @@
             <collision>
                 <geometry>
-                    <mesh filename="${path_to_hip}" scale = "0.001 0.001 0.001"/>
+                    <mesh filename="${path_to_leg_roll}" scale = "0.001 0.001 0.001"/>
                 </geometry>
                 <origin xyz="0.0 0.0 0.0" rpy="${pi/2} 0.0 ${pi*side/2}"/>
             </collision>
         </link>
-        <gazebo reference="${leg}_hip">
+        <gazebo reference="${leg}_leg_roll">
             <material>Gazebo/Orange</material>
         </gazebo>
@@ -100,5 +100,5 @@
         <joint name="${leg}_hip_joint" type="revolute">
             <parent link="base_link"/>
-            <child link="${leg}_hip"/>
+            <child link="${leg}_leg_roll"/>
             <axis xyz="1.0 0.0 0.0"/>
             <origin xyz="${position_hip} 0.0 0.0"/>
@@ -107,5 +107,5 @@
         </joint>
         <joint name="${leg}_upper_leg_joint" type="revolute">
-            <parent link="${leg}_hip"/>
+            <parent link="${leg}_leg_roll"/>
             <child link="${leg}_upper_leg"/>
             <axis xyz="0.0 1.0  0.0"/>

File: src/mini_project/robots/manipulator.urdf.xacro (robot description, xacro)
@@ -2,20 +2,20 @@
 <robot xmlns:xacro="http://www.ros.org/wiki/xacro">
     <xacro:macro name="manipulator" params="base_name">
-        <link name="manipulator_joint">
+        <link name="manipulator_base">
             <inertial>
-                <origin xyz="${man_joint_center}" />
-                <mass value="${man_joint_mass}" />
-                <inertia ixx="${ixx_man_joint}" ixy="${ixy_man_joint}" ixz="${ixz_man_joint}"
-                        iyy="${iyy_man_joint}" iyz="${iyz_man_joint}"
-                        izz="${izz_man_joint}" />
+                <origin xyz="${man_base_center}" />
+                <mass value="${man_base_mass}" />
+                <inertia ixx="${ixx_man_base}" ixy="${ixy_man_base}" ixz="${ixz_man_base}"
+                        iyy="${iyy_man_base}" iyz="${iyz_man_base}"
+                        izz="${izz_man_base}" />
             </inertial>
             <visual>
                 <geometry>
-                    <mesh filename="${path_to_manipulator_joint}" scale = "0.001 0.001 0.001"/>
+                    <mesh filename="${path_to_manipulator_base}" scale = "0.001 0.001 0.001"/>
                 </geometry>
             </visual>
             <collision>
                 <geometry>
-                    <mesh filename="${path_to_manipulator_joint}" scale = "0.001 0.001 0.001"/>
+                    <mesh filename="${path_to_manipulator_base}" scale = "0.001 0.001 0.001"/>
                 </geometry>
             </collision>
@@ -63,11 +63,11 @@
             </collision>
         </link>
-        <joint name="${base_name}_to_manipulator_joint" type="fixed">
+        <joint name="${base_name}_to_manipulator_base" type="fixed">
             <parent link="${base_name}"/>
-            <child link="manipulator_joint"/>
+            <child link="manipulator_base"/>
             <origin xyz="0.0 0.0 0.13"/>
         </joint>
-        <joint name="manipulator_joint_to_manipulator_segment_1" type="fixed">
-            <parent link="manipulator_joint"/>
+        <joint name="manipulator_base_to_manipulator_segment_1" type="fixed">
+            <parent link="manipulator_base"/>
             <child link="manipulator_segment_1"/>
             <origin xyz="0.0 0.04 0.075" rpy="0 0 0"/>

File: src/mini_project/robots/robot_properties.urdf.xacro (robot description, xacro)
@@ -2,8 +2,8 @@
 <robot xmlns:xacro="http://www.ros.org/wiki/xacro">
     <xacro:property name="path_to_base" value = "package://mini_project/meshes/body.dae"/>
-    <xacro:property name="path_to_hip" value = "package://mini_project/meshes/thigh.dae"/>
+    <xacro:property name="path_to_leg_roll" value = "package://mini_project/meshes/thigh.dae"/>
     <xacro:property name="path_to_upper_leg" value = "package://mini_project/meshes/upper_leg.dae"/>
     <xacro:property name="path_to_lower_leg" value = "package://mini_project/meshes/lower_leg.dae"/>
-    <xacro:property name="path_to_manipulator_joint" value = "package://mini_project/meshes/manipulator_joint.dae"/>
+    <xacro:property name="path_to_manipulator_base" value = "package://mini_project/meshes/manipulator_joint.dae"/>
     <xacro:property name="path_to_manipulator_segment_1" value = "package://mini_project/meshes/manipulator_segment_1.dae"/>
     <xacro:property name="path_to_manipulator_segment_2" value = "package://mini_project/meshes/manipulator_segment_2.dae"/>
@@ -16,14 +16,14 @@
     <xacro:property name="body_mass" value = "44.88560358"/>
     <xacro:property name="body_center_of_mass" value = "0 0 -0.00722624877"/>
-    <xacro:property name="ixx_hip" value = "0.01771591024568"/>
-    <xacro:property name="ixy_hip" value = "-0.00071891013320"/>
-    <xacro:property name="ixz_hip" value = "0.00000000005151"/>
-    <xacro:property name="iyy_hip" value = "0.00540298667217"/>
-    <xacro:property name="iyz_hip" value = "0.00000000016635"/>
-    <xacro:property name="izz_hip" value = "0.01761332943090"/>
-    <xacro:property name="hip_mass" value = "2.33840380"/>
-    <xacro:property name="hip_center_x" value = "0.00160346990"/>
-    <xacro:property name="hip_center_y" value = "0.19560047521"/>
-    <xacro:property name="hip_center_z" value = "0.0"/>
+    <xacro:property name="ixx_leg_roll" value = "0.01771591024568"/>
+    <xacro:property name="ixy_leg_roll" value = "-0.00071891013320"/>
+    <xacro:property name="ixz_leg_roll" value = "0.00000000005151"/>
+    <xacro:property name="iyy_leg_roll" value = "0.00540298667217"/>
+    <xacro:property name="iyz_leg_roll" value = "0.00000000016635"/>
+    <xacro:property name="izz_leg_roll" value = "0.01761332943090"/>
+    <xacro:property name="leg_roll_mass" value = "2.33840380"/>
+    <xacro:property name="leg_roll_center_x" value = "0.00160346990"/>
+    <xacro:property name="leg_roll_center_y" value = "0.19560047521"/>
+    <xacro:property name="leg_roll_center_z" value = "0.0"/>
     <xacro:property name="ixx_thigh" value = "0.07057863"/>
     <xacro:property name="ixy_thigh" value = "0.0"/>
@@ -48,12 +48,12 @@
     <xacro:property name="lower_leg_center_z" value = "-0.15457863"/>
     <xacro:property name="lower_leg_center_of_mass" value = "${lower_leg_center_x} ${lower_leg_center_y} ${lower_leg_center_z}"/>
-    <xacro:property name="ixx_man_joint" value = "0.00592368152307"/>
-    <xacro:property name="ixy_man_joint" value = "-0.00000002959529"/>
-    <xacro:property name="ixz_man_joint" value = "0.00000000508195"/>
-    <xacro:property name="iyy_man_joint" value = "0.00455222665474"/>
-    <xacro:property name="iyz_man_joint" value = "-0.00046066688062"/>
-    <xacro:property name="izz_man_joint" value = "0.00630165344962"/>
-    <xacro:property name="man_joint_mass" value = "1.63291158"/>
-    <xacro:property name="man_joint_center" value = "0.0001195 -0.01132600777 0.04996291284 "/>
+    <xacro:property name="ixx_man_base" value = "0.00592368152307"/>
+    <xacro:property name="ixy_man_base" value = "-0.00000002959529"/>
+    <xacro:property name="ixz_man_base" value = "0.00000000508195"/>
+    <xacro:property name="iyy_man_base" value = "0.00455222665474"/>
+    <xacro:property name="iyz_man_base" value = "-0.00046066688062"/>
+    <xacro:property name="izz_man_base" value = "0.00630165344962"/>
+    <xacro:property name="man_base_mass" value = "1.63291158"/>
+    <xacro:property name="man_base_center" value = "0.0001195 -0.01132600777 0.04996291284 "/>
     <xacro:property name="ixx_man_seg_1" value = "0.00029149081721"/>
     <xacro:property name="ixy_man_seg_1" value = "0.00000011029091"/>
