Commit message: adding 3 zed cameras

File: src/mini_project/robots/husky/husky.urdf.xacro (robot description, xacro)
@@ -205,5 +205,8 @@
     </xacro:vlp16_mount>
   </xacro:if>
-  <xacro:zed_camera base_name = "base_link"/>
+  <xacro:zed_camera base_name="base_link" pos_x="0.15" pos_y="0.0" pos_z="0.5" rotate_camera="0.0" camera_numb="1"/>
+  <xacro:zed_camera base_name="base_link" pos_x="0.0" pos_y="-0.15" pos_z="0.5" rotate_camera="0.5" camera_numb="2"/>
+  <xacro:zed_camera base_name="base_link" pos_x="0.0" pos_y="0.15" pos_z="0.5" rotate_camera="-0.5" camera_numb="3"/>
+  <xacro:zed_camera base_name="base_link" pos_x="-0.15" pos_y="0.0" pos_z="0.5" rotate_camera="1" camera_numb="4"/>
   <gazebo>
     <plugin name="gazebo_ros_control" filename="libgazebo_ros_control.so">

File: src/mini_project/robots/husky/zed_camera.urdf.xacro (robot description, xacro)
@@ -1,19 +1,33 @@
 <?xml version="1.0"?>
 <robot xmlns:xacro="http://ros.org/wiki/xacro">
-    <xacro:macro name="zed_camera" params="base_name " >
-    <xacro:include filename="$(find mini_project)/robots/materials.urdf.xacro" />
+    <xacro:macro name="zed_camera" params="base_name pos_x pos_y pos_z rotate_camera camera_numb" >
     <!-- Arguments -->
     <xacro:arg name="camera_name"   default="zed2" />
     <xacro:arg name="camera_model"  default="zed2" />
     <xacro:arg name="base_frame"    default="${base_name}" />
-    <xacro:arg name="cam_pos_x"     default="0.495" />
-    <xacro:arg name="cam_pos_y"     default="0.0" />
-    <xacro:arg name="cam_pos_z"     default="0.09" />
     <xacro:arg name="cam_roll"      default="0.0" />
     <xacro:arg name="cam_pitch"     default="0.0" />
     <xacro:arg name="cam_yaw"       default="0.0" />
     <!-- Properties -->
-    <xacro:property name="M_PI"     value="3.1415926535897931" />
-    <xacro:property name="model"    value="$(arg camera_model)" />
+    <xacro:property name="M_PI"          value="3.1415926535897931" />
+    <xacro:property name="model"         value="$(arg camera_model)" />
+    <xacro:property name="cam_pos_x"     value="${pos_x}" />
+    <xacro:property name="cam_pos_y"     value="${pos_y}" />
+    <xacro:property name="cam_pos_z"     value="${pos_z}" />
+    <xacro:property name="rotate"        value="${rotate_camera}" />
+    <xacro:property name="numb"          value="${camera_numb}" />
+    <!-- Materials -->
+    <material name="zed_mat_${numb}">
+        <color rgba="0.8 0.8 0.8 0.8"/>
+    </material>
+    <material name="zedm_mat_${numb}">
+        <color rgba="0 0 0 0.9"/>
+    </material>
+    <material name="zed2_mat_${numb}">
+        <color rgba="0.25 0.25 0.25 0.99"/>
+    </material>
+    <material name="zed2i_mat_${numb}">
+        <color rgba="0.25 0.25 0.25 0.99"/>
+    </material>
     <xacro:if value="${model == 'zed'}">
         <xacro:property name="baseline" value="0.12" />
@@ -29,32 +43,32 @@
     </xacro:if>
 <!-- Camera Center -->
-    <joint name="camera_center_joint" type="fixed">
+    <joint name="camera_center_joint_${numb}" type="fixed">
         <parent link="$(arg base_frame)"/>
-        <child link="camera_center"/>
-        <origin xyz="$(arg cam_pos_x) $(arg cam_pos_y) $(arg cam_pos_z)" rpy="$(arg cam_roll) $(arg cam_pitch) $(arg cam_yaw)" />
+        <child link="camera_center_${numb}"/>
+        <origin xyz="${cam_pos_x} ${cam_pos_y} ${cam_pos_z}" rpy="$(arg cam_roll) $(arg cam_pitch) $(arg cam_yaw)" />
     </joint>
-    <link name="camera_center">
+    <link name="camera_center_${numb}">
         <visual>
-            <origin xyz="0 0 0" rpy="0 0 0"/>
+            <origin xyz="0 0 0" rpy="0 0 ${rotate*M_PI}"/>
             <geometry>
                 <mesh filename="package://mini_project/meshes/${model}.stl" />
             </geometry>
-            <material name="${model}_mat" />
+            <material name="${model}_mat_${numb}" />
         </visual>
     </link>
 <!-- Left Camera -->
-    <joint name="left_camera_joint" type="fixed">
-        <parent link="camera_center"/>
-        <child link="left_camera_frame"/>
+    <joint name="left_camera_joint_${numb}" type="fixed">
+        <parent link="camera_center_${numb}"/>
+        <child link="left_camera_frame_${numb}"/>
         <origin xyz="0 ${baseline/2} 0" rpy="0 0 0" />
     </joint>
-    <link name="left_camera_frame" />
-    <joint name="left_camera_optical_joint" type="fixed">
+    <link name="left_camera_frame_${numb}" />
+    <joint name="left_camera_optical_joint_${numb}" type="fixed">
         <origin xyz="0 0 0" rpy="-${M_PI/2} 0.0 -${M_PI/2}"/>
-        <parent link="left_camera_frame"/>
-        <child link="left_camera_optical_frame"/>
+        <parent link="left_camera_frame_${numb}"/>
+        <child link="left_camera_optical_frame_${numb}"/>
     </joint>
-    <link name="left_camera_optical_frame"/>
-    <gazebo reference="left_camera_frame">
+    <link name="left_camera_optical_frame_${numb}"/>
+    <gazebo reference="left_camera_frame_${numb}">
         <sensor type="multicamera" name="stereo_camera">
         <update_rate>30.0</update_rate>
@@ -102,8 +116,8 @@
             <alwaysOn>true</alwaysOn>
             <updateRate>0.0</updateRate>
-            <cameraName>camera</cameraName>
+            <cameraName>camera_${numb}</cameraName>
             <imageTopicName>image_raw</imageTopicName>
             <cameraInfoTopicName>camera_info</cameraInfoTopicName>
-            <frameName>left_camera_optical_frame</frameName>
+            <frameName>left_camera_optical_frame_${numb}</frameName>
             <!--<rightFrameName>right_camera_optical_frame</rightFrameName>-->
             <hackBaseline>0.12</hackBaseline>

Commit message: disp/point to laserscan for husky

File: src/mini_project/robots/husky/husky.urdf.xacro (robot description, xacro)
@@ -55,4 +55,6 @@
   <xacro:arg name="urdf_extras" default="$(optenv HUSKY_URDF_EXTRAS empty.urdf)" />
   <xacro:arg name="cpr_urdf_extras" default="$(optenv CPR_URDF_EXTRAS empty.urdf)" />
+  <!-- four cameras -->
+  <xacro:arg name="four_cameras" default="false" />
   <!-- Included URDF/XACRO Files -->
   <xacro:include filename="$(find husky_description)/urdf/decorations.urdf.xacro" />
@@ -206,7 +208,9 @@
   </xacro:if>
   <xacro:zed_camera base_name="base_link" pos_x="0.15" pos_y="0.0" pos_z="0.5" rotate_camera="0.0" camera_numb="1"/>
-  <xacro:zed_camera base_name="base_link" pos_x="0.0" pos_y="-0.15" pos_z="0.5" rotate_camera="0.5" camera_numb="2"/>
-  <xacro:zed_camera base_name="base_link" pos_x="0.0" pos_y="0.15" pos_z="0.5" rotate_camera="-0.5" camera_numb="3"/>
-  <xacro:zed_camera base_name="base_link" pos_x="-0.15" pos_y="0.0" pos_z="0.5" rotate_camera="1" camera_numb="4"/>
+  <xacro:if value="$(arg four_cameras)">
+    <xacro:zed_camera base_name="base_link" pos_x="0.0" pos_y="-0.15" pos_z="0.5" rotate_camera="0.5" camera_numb="2"/>
+    <xacro:zed_camera base_name="base_link" pos_x="0.0" pos_y="0.15" pos_z="0.5" rotate_camera="-0.5" camera_numb="3"/>
+    <xacro:zed_camera base_name="base_link" pos_x="-0.15" pos_y="0.0" pos_z="0.5" rotate_camera="1.0" camera_numb="4"/>
+  </xacro:if>
   <gazebo>
     <plugin name="gazebo_ros_control" filename="libgazebo_ros_control.so">

File: src/mini_project/robots/husky/zed_camera.urdf.xacro (robot description, xacro)
@@ -46,9 +46,9 @@
         <parent link="$(arg base_frame)"/>
         <child link="camera_center_${numb}"/>
-        <origin xyz="${cam_pos_x} ${cam_pos_y} ${cam_pos_z}" rpy="$(arg cam_roll) $(arg cam_pitch) $(arg cam_yaw)" />
+        <origin xyz="${cam_pos_x} ${cam_pos_y} ${cam_pos_z}" rpy="$(arg cam_roll) $(arg cam_pitch) ${rotate*M_PI}" />
     </joint>
     <link name="camera_center_${numb}">
         <visual>
-            <origin xyz="0 0 0" rpy="0 0 ${rotate*M_PI}"/>
+            <origin xyz="0 0 0" rpy="0 0 0"/>
             <geometry>
                 <mesh filename="package://mini_project/meshes/${model}.stl" />

Commit message: stereo orbslam

File: src/mini_project/robots/husky/husky.urdf.xacro (robot description, xacro)
@@ -121,12 +121,16 @@
   <!-- IMU Link is the standard mounting position for the UM6 IMU.-->
   <!-- Can be modified with environment variables in /etc/ros/setup.bash -->
-  <link name="imu_link"/>
+  <link name="imu_link">
+      <inertial>
+          <mass value="0.001"/>
+          <origin xyz="0 0 0" rpy="0 0 0"/>
+          <inertia ixx="1e-09" ixy="0.0" ixz="0.0" iyy="1e-09" iyz="0.0" izz="1e-09"/>
+      </inertial>
+  </link>
   <joint name="imu_joint" type="fixed">
-    <origin xyz="$(optenv HUSKY_IMU_XYZ 0.19 0 0.149)" rpy="$(optenv HUSKY_IMU_RPY 0 -1.5708 3.1416)" />
-    <parent link="base_link" />
-    <child link="imu_link" />
+      <parent link="base_link" />
+      <child link="imu_link" />
+      <origin xyz="0.15 0 0.5" rpy="0 0 0"/>
   </joint>
-  <gazebo reference="imu_link">
-  </gazebo>
   <!-- Husky wheel macros -->
   <xacro:husky_wheel wheel_prefix="front_left">
@@ -225,10 +229,10 @@
       <bodyName>base_link</bodyName>
       <topicName>imu/data</topicName>
-      <accelDrift>0.000 0.000 0.000</accelDrift>
-      <accelGaussianNoise>0.000 0.000 0.000</accelGaussianNoise>
-      <rateDrift>0.000 0.000 0.000 </rateDrift>
-      <rateGaussianNoise>0.000 0.000 0.000 </rateGaussianNoise>
-      <headingDrift>0.000</headingDrift>
-      <headingGaussianNoise>0.000</headingGaussianNoise>
+      <accelDrift>0.005 0.005 0.005</accelDrift>
+      <accelGaussianNoise>0.005 0.005 0.005</accelGaussianNoise>
+      <rateDrift>0.005 0.005 0.005 </rateDrift>
+      <rateGaussianNoise>0.005 0.005 0.005 </rateGaussianNoise>
+      <headingDrift>0.005</headingDrift>
+      <headingGaussianNoise>0.005</headingGaussianNoise>
     </plugin>
   </gazebo>

File: src/mini_project/robots/husky/zed_camera.urdf.xacro (robot description, xacro)
@@ -70,7 +70,19 @@
     </joint>
     <link name="left_camera_optical_frame_${numb}"/>
+    <joint name="right_camera_joint_${numb}" type="fixed">
+        <parent link="camera_center_${numb}"/>
+        <child link="right_camera_frame_${numb}"/>
+        <origin xyz="0 -${baseline/2} 0" rpy="0 0 0" />
+    </joint>
+    <link name="right_camera_frame_${numb}" />
+    <joint name="right_camera_optical_joint_${numb}" type="fixed">
+        <origin xyz="0 0 0" rpy="-${M_PI/2} 0.0 -${M_PI/2}"/>
+        <parent link="right_camera_frame_${numb}"/>
+        <child link="right_camera_optical_frame_${numb}"/>
+    </joint>
+    <link name="right_camera_optical_frame_${numb}"/>
     <gazebo reference="left_camera_frame_${numb}">
         <sensor type="multicamera" name="stereo_camera">
-        <update_rate>30.0</update_rate>
+        <update_rate>20.0</update_rate>
         <camera name="left">
             <horizontal_fov>1.91986218</horizontal_fov>
@@ -86,9 +98,4 @@
                 <far>300</far>
             </clip>
-            <noise>
-                <type>gaussian</type>
-                <mean>0.0</mean>
-                <stddev>0.004</stddev>
-            </noise>
         </camera>
         <camera name="right">
@@ -106,9 +113,4 @@
                 <far>300</far>
             </clip>
-            <noise>
-                <type>gaussian</type>
-                <mean>0.0</mean>
-                <stddev>0.004</stddev>
-            </noise>
         </camera>
         <plugin name="stereo_camera_controller" filename="libgazebo_ros_multicamera.so">

Commit message: change camera sub (camera-imu)

File: src/mini_project/robots/husky/husky.urdf.xacro (robot description, xacro)
@@ -131,5 +131,5 @@
       <parent link="base_link" />
       <child link="imu_link" />
-      <origin xyz="0.15 0 0.5" rpy="0 0 0"/>
+      <origin xyz="0.0 0 0.0" rpy="-1.57079632679 0 -1.57079632679"/>
   </joint>
   <!-- Husky wheel macros -->
@@ -226,6 +226,7 @@
     <plugin name="imu_controller" filename="libhector_gazebo_ros_imu.so">
       <robotNamespace>$(arg robot_namespace)</robotNamespace>
-      <updateRate>400.0</updateRate>
-      <bodyName>base_link</bodyName>
+      <always_on>1</always_on>
+      <updateRate>200.0</updateRate>
+      <bodyName>imu_link</bodyName>
       <topicName>imu/data</topicName>
       <accelDrift>0.005 0.005 0.005</accelDrift>

Commit message: change husky imu urdf

File: src/mini_project/robots/husky/husky.urdf.xacro (robot description, xacro)
@@ -131,5 +131,5 @@
       <parent link="base_link" />
       <child link="imu_link" />
-      <origin xyz="0.0 0 0.0" rpy="-1.57079632679 0 -1.57079632679"/>
+      <origin xyz="0.0 0 0.0" rpy="0.0 0.0 0.0"/>
   </joint>
   <!-- Husky wheel macros -->
@@ -230,10 +230,10 @@
       <bodyName>imu_link</bodyName>
       <topicName>imu/data</topicName>
-      <accelDrift>0.005 0.005 0.005</accelDrift>
-      <accelGaussianNoise>0.005 0.005 0.005</accelGaussianNoise>
-      <rateDrift>0.005 0.005 0.005 </rateDrift>
-      <rateGaussianNoise>0.005 0.005 0.005 </rateGaussianNoise>
-      <headingDrift>0.005</headingDrift>
-      <headingGaussianNoise>0.005</headingGaussianNoise>
+      <accelDrift>0.001 0.001 0.001</accelDrift>
+      <accelGaussianNoise>0.001 0.001 0.001</accelGaussianNoise>
+      <rateDrift>0.001 0.001 0.001 </rateDrift>
+      <rateGaussianNoise>0.001 0.001 0.001 </rateGaussianNoise>
+      <headingDrift>0.001</headingDrift>
+      <headingGaussianNoise>0.001</headingGaussianNoise>
     </plugin>
   </gazebo>

File: src/mini_project/robots/husky/zed_camera.urdf.xacro (robot description, xacro)
@@ -84,5 +84,5 @@
     <gazebo reference="left_camera_frame_${numb}">
         <sensor type="multicamera" name="stereo_camera">
-        <update_rate>30.0</update_rate>
+        <update_rate>15.0</update_rate>
         <camera name="left">
             <horizontal_fov>1.91986218</horizontal_fov>
